File: xmosxl.sch (EAGLE design)
At the start: 123 parts, among them IC1 74LVC1T45W6-7, IC2 74LVC1T45W6-7, IC3 74LVC1T45W6-7, IC4 74LVC1T45W6-7, IC5 74LVC1T45W6-7, IC6 74ALVC164245DGG_11, IC7 74ALVC164245DGG_11, IC8 74LVC1T45W6-7, IC9 74LVC1T45W6-7, U1 24 MHz Osc. (F535L-24)

Commit message: Add the links
Parts:
- added C59, C60, C61, C62, C63, C64, C65, C66: 100nF, rcl:C-EUC0201
- added I2C0, I2C1: (no value), pinhead:PINHD-1X2
- added JP1: (no value), pinhead:PINHD-2X9
- added R27, R28: 43R2, rcl:R-EU_R0201
- added R29, R30: 4K7, rcl:R-EU_R0201
- added R31, R32, R33, R34, R35: 33R, rcl:R-EU_R0201
- added UART: (no value), pinhead:PINHD-1X3
Connections:
- new net N$11: R27.2, XMOS-USB.USB_RTUNE_1@W16
- new net N$12: R28.2, XMOS-USB.USB_RTUNE_0@W6
- new net N$13: UART.2, XMOS-UART.X1D35@E3
- new net N$20: UART.1, XMOS-UART.X1D34@D3
- new net N$21: JP1.4
- new net N$24: JP1.8
- new net N$25: JP1.12
- new net N$26: JP1.16
- new net N$27: R31.1, XMOS-LINK.X1D66@N2
- new net N$28: R32.1, XMOS-LINK.X1D67@P2
- new net N$29: R34.1, XMOS-LINK.X1D69@R1
- new net N$30: R35.1, XMOS-LINK.X1D70@R2
- new net RX0: JP1.1, XMOS-LINK.X1D65@N1
- new net RX1: JP1.5, XMOS-LINK.X1D64@M1
- new net RX2: JP1.9, XMOS-LINK.X1D63@M2
- new net RX3: JP1.13, XMOS-LINK.X1D62@M3
- new net RX4: JP1.17, R33.1, XMOS-LINK.X1D61@L3, XMOS-LINK.X1D68@P1
- new net SCL: I2C0.1, I2C1.1, R29.1, XMOS-I2C.X1D11@A3
- new net SDA: I2C0.2, I2C1.2, R30.1, XMOS-I2C.X1D10@B3
- new net TX0: JP1.2, R31.2
- new net TX1: JP1.6, R32.2
- new net TX2: JP1.10, R33.2
- new net TX3: JP1.14, R34.2
- new net TX4: JP1.18, R35.2
- net +3V3: now also C59.1, C60.1, C61.1, C62.1, C63.1, C64.1, C65.1, C66.1, JP1.11, R29.2, R30.2
- net +5V: now also JP1.7
- net GND: now also C59.2, C60.2, C61.2, C62.2, C63.2, C64.2, C65.2, C66.2, JP1.3, R27.1, R28.1, UART.3
- net VDD: now also JP1.15
Other:
- note added: "Atari Interface / Level Converters"
- note added: "Block diagram"
- note added: "Clock, Jtag, USB, Leds and Reset"
- note added: "SDRAM to XMOS"
- note added: "XMOS Power in"
- note added: "XMOS to Atari, I2C and UART"
- note removed: "3.3v from +5v"
- note removed: "Gated 1v from +5v"
- note removed: "Power entry"
- moved on the sheet: C21, C22, C23, C24, C25, C26, C27, C28, C29, C30, C31, C32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
